File: switch-matrix/switch-matrix.kicad_pcb (KiCad board)
At the start: 2 copper layers, 245 parts, among them IC301 ATMEGA328P-A, P101 USB_OTG, P102 CONN_01X04, P301 CONN_01X06, Q1701 BSS84, Q1702 MMBT3904, Q1703 MMBT3904, Q1801 BSS84, Q1802 MMBT3904, Q1803 MMBT3904, Q1901 BSS84, Q1902 MMBT3904, Q1903 MMBT3904, U201 ST662AC, U401 FMS6501A, U402 FMS6501A, U403 FMS6501A, U404 FMS6501A, U405 FMS6501A, U406 FMS6501A

Commit message: + Add the dual LED footprint. * Got the input scart connector grid sorted with a little layout duplication script.
Parts:
- removed R419, R420, R421, R422, R423, R424: 75, Capacitors_SMD:C_0603
- added D301: LED_BI, scart:0605LEDDual, F.Cu at (606.1, 189.2)
- added JP1001: Jumper_NO_Small, Connect:GS2, B.Cu at (73.0, 141.8)
- added JP1002: Jumper_NC_Small, Connect:GS2, B.Cu at (82.8, 139.8)
- added JP1003: Jumper_NO_Small, Connect:GS2, B.Cu at (73.0, 137.9)
- added JP1004: Jumper_NC_Small, Connect:GS2, B.Cu at (82.8, 132.2)
- added JP1005: Jumper_NO_Small, Connect:GS2, B.Cu at (73.0, 107.4)
- added JP1006: Jumper_NC_Small, Connect:GS2, B.Cu at (82.8, 105.5)
- added JP1101: Jumper_NO_Small, Connect:GS2, B.Cu at (98.0, 73.8)
- added JP1102: Jumper_NC_Small, Connect:GS2, B.Cu at (107.8, 71.8)
- added JP1103: Jumper_NO_Small, Connect:GS2, B.Cu at (98.0, 69.9)
- added JP1104: Jumper_NC_Small, Connect:GS2, B.Cu at (107.8, 64.2)
- added JP1105: Jumper_NO_Small, Connect:GS2, B.Cu at (98.0, 39.4)
- added JP1106: Jumper_NC_Small, Connect:GS2, B.Cu at (107.8, 37.5)
- added JP1201: Jumper_NO_Small, Connect:GS2, B.Cu at (98.0, 141.8)
- added JP1202: Jumper_NC_Small, Connect:GS2, B.Cu at (107.8, 139.8)
- added JP1203: Jumper_NO_Small, Connect:GS2, B.Cu at (98.0, 137.9)
- added JP1204: Jumper_NC_Small, Connect:GS2, B.Cu at (107.8, 132.2)
- added JP1205: Jumper_NO_Small, Connect:GS2, B.Cu at (98.0, 107.4)
- added JP1206: Jumper_NC_Small, Connect:GS2, B.Cu at (107.8, 105.5)
- added JP1301: Jumper_NO_Small, Connect:GS2, B.Cu at (123.0, 73.8)
- added JP1302: Jumper_NC_Small, Connect:GS2, B.Cu at (132.8, 71.8)
- added JP1303: Jumper_NO_Small, Connect:GS2, B.Cu at (123.0, 69.9)
- added JP1304: Jumper_NC_Small, Connect:GS2, B.Cu at (132.8, 64.2)
- added JP1305: Jumper_NO_Small, Connect:GS2, B.Cu at (123.0, 39.4)
- added JP1306: Jumper_NC_Small, Connect:GS2, B.Cu at (132.8, 37.5)
- added JP1401: Jumper_NO_Small, Connect:GS2, B.Cu at (123.0, 141.8)
- added JP1402: Jumper_NC_Small, Connect:GS2, B.Cu at (132.8, 139.8)
- added JP1403: Jumper_NO_Small, Connect:GS2, B.Cu at (123.0, 137.9)
- added JP1404: Jumper_NC_Small, Connect:GS2, B.Cu at (132.8, 132.2)
- added JP1405: Jumper_NO_Small, Connect:GS2, B.Cu at (123.0, 107.4)
- added JP1406: Jumper_NC_Small, Connect:GS2, B.Cu at (132.8, 105.5)
- added JP1501: Jumper_NO_Small, Connect:GS2, B.Cu at (148.0, 73.8)
- added JP1502: Jumper_NC_Small, Connect:GS2, B.Cu at (157.8, 71.8)
- added JP1503: Jumper_NO_Small, Connect:GS2, B.Cu at (148.0, 69.9)
- added JP1504: Jumper_NC_Small, Connect:GS2, B.Cu at (157.8, 64.2)
- added JP1505: Jumper_NO_Small, Connect:GS2, B.Cu at (148.0, 39.4)
- added JP1506: Jumper_NC_Small, Connect:GS2, B.Cu at (157.8, 37.5)
- added JP1601: Jumper_NO_Small, Connect:GS2, B.Cu at (148.0, 141.8)
- added JP1602: Jumper_NC_Small, Connect:GS2, B.Cu at (157.8, 139.8)
- added JP1603: Jumper_NO_Small, Connect:GS2, B.Cu at (148.0, 137.9)
- added JP1604: Jumper_NC_Small, Connect:GS2, B.Cu at (157.8, 132.2)
- added JP1605: Jumper_NO_Small, Connect:GS2, B.Cu at (148.0, 107.4)
- added JP1606: Jumper_NC_Small, Connect:GS2, B.Cu at (157.8, 105.5)
- added JP501: Jumper_NO_Small, Connect:GS2, B.Cu at (23.0, 73.8)
- added JP502: Jumper_NC_Small, Connect:GS2, B.Cu at (32.8, 71.8)
- added JP503: Jumper_NO_Small, Connect:GS2, B.Cu at (23.0, 69.9)
- added JP504: Jumper_NC_Small, Connect:GS2, B.Cu at (32.8, 64.2)
- added JP505: Jumper_NO_Small, Connect:GS2, B.Cu at (23.0, 39.4)
- added JP506: Jumper_NC_Small, Connect:GS2, B.Cu at (32.8, 37.5)
- added JP601: Jumper_NO_Small, Connect:GS2, B.Cu at (23.0, 141.8)
- added JP602: Jumper_NC_Small, Connect:GS2, B.Cu at (32.8, 139.8)
- added JP603: Jumper_NO_Small, Connect:GS2, B.Cu at (23.0, 137.9)
- added JP604: Jumper_NC_Small, Connect:GS2, B.Cu at (32.8, 132.2)
- added JP605: Jumper_NO_Small, Connect:GS2, B.Cu at (23.0, 107.4)
- added JP606: Jumper_NC_Small, Connect:GS2, B.Cu at (32.8, 105.5)
- added JP701: Jumper_NO_Small, Connect:GS2, B.Cu at (48.0, 73.8)
- added JP702: Jumper_NC_Small, Connect:GS2, B.Cu at (57.8, 71.8)
- added JP703: Jumper_NO_Small, Connect:GS2, B.Cu at (48.0, 69.9)
- added JP704: Jumper_NC_Small, Connect:GS2, B.Cu at (57.8, 64.2)
- added JP705: Jumper_NO_Small, Connect:GS2, B.Cu at (48.0, 39.4)
- added JP706: Jumper_NC_Small, Connect:GS2, B.Cu at (57.8, 37.5)
- added JP801: Jumper_NO_Small, Connect:GS2, B.Cu at (48.0, 141.8)
- added JP802: Jumper_NC_Small, Connect:GS2, B.Cu at (57.8, 139.8)
- added JP803: Jumper_NO_Small, Connect:GS2, B.Cu at (48.0, 137.9)
- added JP804: Jumper_NC_Small, Connect:GS2, B.Cu at (57.8, 132.2)
- added JP805: Jumper_NO_Small, Connect:GS2, B.Cu at (48.0, 107.4)
- added JP806: Jumper_NC_Small, Connect:GS2, B.Cu at (57.8, 105.5)
- added JP901: Jumper_NO_Small, Connect:GS2, B.Cu at (73.0, 73.8)
- added JP902: Jumper_NC_Small, Connect:GS2, B.Cu at (82.8, 71.8)
- added JP903: Jumper_NO_Small, Connect:GS2, B.Cu at (73.0, 69.9)
- added JP904: Jumper_NC_Small, Connect:GS2, B.Cu at (82.8, 64.2)
- added JP905: Jumper_NO_Small, Connect:GS2, B.Cu at (73.0, 39.4)
- added JP906: Jumper_NC_Small, Connect:GS2, B.Cu at (82.8, 37.5)
- added L201: 100u, Inductors_NEOSID:Neosid_Inductor_SM-NE127, F.Cu at (596.5, 158.7)
- added L202: 100u, Inductors_NEOSID:Neosid_Inductor_SM-NE127, F.Cu at (609.7, 158.7)
- added L203: 100u, Inductors_NEOSID:Neosid_Inductor_SM-NE127, F.Cu at (622.9, 158.7)
- added R1005: 10k, Resistors_SMD:R_0603, B.Cu at (84.2, 141.8)
- added R1006: 10k, Resistors_SMD:R_0603, B.Cu at (83.0, 136.9)
- added R1007: 75, Capacitors_SMD:C_0603, B.Cu at (73.3, 132.6)
- added R1008: 75, Capacitors_SMD:C_0603, B.Cu at (73.3, 125.0)
- added R1009: 75, Capacitors_SMD:C_0603, B.Cu at (73.3, 117.4)
- added R1010: 75, Capacitors_SMD:C_0603, B.Cu at (81.1, 102.2)
- added R1105: 10k, Resistors_SMD:R_0603, B.Cu at (109.2, 73.8)
- added R1106: 10k, Resistors_SMD:R_0603, B.Cu at (108.0, 68.9)
- added R1107: 75, Capacitors_SMD:C_0603, B.Cu at (98.3, 64.6)
- added R1108: 75, Capacitors_SMD:C_0603, B.Cu at (98.3, 57.0)
- added R1109: 75, Capacitors_SMD:C_0603, B.Cu at (98.3, 49.4)
- added R1110: 75, Capacitors_SMD:C_0603, B.Cu at (106.1, 34.2)
- added R1205: 10k, Resistors_SMD:R_0603, B.Cu at (109.2, 141.8)
- added R1206: 10k, Resistors_SMD:R_0603, B.Cu at (108.0, 136.9)
- added R1207: 75, Capacitors_SMD:C_0603, B.Cu at (98.3, 132.6)
- added R1208: 75, Capacitors_SMD:C_0603, B.Cu at (98.3, 125.0)
- added R1209: 75, Capacitors_SMD:C_0603, B.Cu at (98.3, 117.4)
- added R1210: 75, Capacitors_SMD:C_0603, B.Cu at (106.1, 102.2)
- added R1305: 10k, Resistors_SMD:R_0603, B.Cu at (134.2, 73.8)
- added R1306: 10k, Resistors_SMD:R_0603, B.Cu at (133.0, 68.9)
- added R1307: 75, Capacitors_SMD:C_0603, B.Cu at (123.3, 64.6)
- added R1308: 75, Capacitors_SMD:C_0603, B.Cu at (123.3, 57.0)
- added R1309: 75, Capacitors_SMD:C_0603, B.Cu at (123.3, 49.4)
- added R1310: 75, Capacitors_SMD:C_0603, B.Cu at (131.1, 34.2)
- added R1405: 10k, Resistors_SMD:R_0603, B.Cu at (134.2, 141.8)
- added R1406: 10k, Resistors_SMD:R_0603, B.Cu at (133.0, 136.9)
- added R1407: 75, Capacitors_SMD:C_0603, B.Cu at (123.3, 132.6)
- added R1408: 75, Capacitors_SMD:C_0603, B.Cu at (123.3, 125.0)
- added R1409: 75, Capacitors_SMD:C_0603, B.Cu at (123.3, 117.4)
- added R1410: 75, Capacitors_SMD:C_0603, B.Cu at (131.1, 102.2)
- added R1505: 10k, Resistors_SMD:R_0603, B.Cu at (159.2, 73.8)
- added R1506: 10k, Resistors_SMD:R_0603, B.Cu at (158.0, 68.9)
- added R1507: 75, Capacitors_SMD:C_0603, B.Cu at (148.3, 64.6)
- added R1508: 75, Capacitors_SMD:C_0603, B.Cu at (148.3, 57.0)
- added R1509: 75, Capacitors_SMD:C_0603, B.Cu at (148.3, 49.4)
- added R1510: 75, Capacitors_SMD:C_0603, B.Cu at (156.1, 34.2)
- added R1605: 10k, Resistors_SMD:R_0603, B.Cu at (159.2, 141.8)
- added R1606: 10k, Resistors_SMD:R_0603, B.Cu at (158.0, 136.9)
- added R1607: 75, Capacitors_SMD:C_0603, B.Cu at (148.3, 132.6)
- added R1608: 75, Capacitors_SMD:C_0603, B.Cu at (148.3, 125.0)
- added R1609: 75, Capacitors_SMD:C_0603, B.Cu at (148.3, 117.4)
- added R1610: 75, Capacitors_SMD:C_0603, B.Cu at (156.1, 102.2)
- added R1704: 10k, Capacitors_SMD:C_0603, F.Cu at (529.8, 97.2)
- added R1705: 10k, Capacitors_SMD:C_0603, F.Cu at (553.8, 90.9)
- added R1804: 10k, Capacitors_SMD:C_0603, F.Cu at (553.8, 133.8)
- added R1805: 10k, Capacitors_SMD:C_0603, F.Cu at (529.8, 140.1)
- added R1904: 10k, Capacitors_SMD:C_0603, F.Cu at (455.4, 183.5)
- added R1905: 10k, Capacitors_SMD:C_0603, F.Cu at (479.4, 177.2)
- added R505: 10k, Resistors_SMD:R_0603, B.Cu at (34.2, 73.8)
- added R506: 10k, Resistors_SMD:R_0603, B.Cu at (33.0, 68.9)
- added R507: 75, Capacitors_SMD:C_0603, B.Cu at (23.3, 64.6)
- added R508: 75, Capacitors_SMD:C_0603, B.Cu at (23.3, 57.0)
- added R509: 75, Capacitors_SMD:C_0603, B.Cu at (23.3, 49.4)
- added R510: 75, Capacitors_SMD:C_0603, B.Cu at (31.1, 34.2)
- added R605: 10k, Resistors_SMD:R_0603, B.Cu at (34.2, 141.8)
- added R606: 10k, Resistors_SMD:R_0603, B.Cu at (33.0, 136.9)
- added R607: 75, Capacitors_SMD:C_0603, B.Cu at (23.3, 132.6)
- added R608: 75, Capacitors_SMD:C_0603, B.Cu at (23.3, 125.0)
- added R609: 75, Capacitors_SMD:C_0603, B.Cu at (23.3, 117.4)
- added R610: 75, Capacitors_SMD:C_0603, B.Cu at (31.1, 102.2)
- added R705: 10k, Resistors_SMD:R_0603, B.Cu at (59.2, 73.8)
- added R706: 10k, Resistors_SMD:R_0603, B.Cu at (58.0, 68.9)
- added R707: 75, Capacitors_SMD:C_0603, B.Cu at (48.3, 64.6)
- added R708: 75, Capacitors_SMD:C_0603, B.Cu at (48.3, 57.0)
- added R709: 75, Capacitors_SMD:C_0603, B.Cu at (48.3, 49.4)
- added R710: 75, Capacitors_SMD:C_0603, B.Cu at (56.1, 34.2)
- added R805: 10k, Resistors_SMD:R_0603, B.Cu at (59.2, 141.8)
- added R806: 10k, Resistors_SMD:R_0603, B.Cu at (58.0, 136.9)
- added R807: 75, Capacitors_SMD:C_0603, B.Cu at (48.3, 132.6)
- added R808: 75, Capacitors_SMD:C_0603, B.Cu at (48.3, 125.0)
- added R809: 75, Capacitors_SMD:C_0603, B.Cu at (48.3, 117.4)
- added R810: 75, Capacitors_SMD:C_0603, B.Cu at (56.1, 102.2)
- added R905: 10k, Resistors_SMD:R_0603, B.Cu at (84.2, 73.8)
- added R906: 10k, Resistors_SMD:R_0603, B.Cu at (83.0, 68.9)
- added R907: 75, Capacitors_SMD:C_0603, B.Cu at (73.3, 64.6)
- added R908: 75, Capacitors_SMD:C_0603, B.Cu at (73.3, 57.0)
- added R909: 75, Capacitors_SMD:C_0603, B.Cu at (73.3, 49.4)
- added R910: 75, Capacitors_SMD:C_0603, B.Cu at (81.1, 34.2)
- C1003, C1004, C1005, C1006, C1103, C1104, C1105, C1106, C1203, C1204, C1205, C1206, C1303, C1304, C1305, C1306, C1403, C1404, C1405, C1406, C1503, C1504, C1505, C1506, C1603, C1604, C1605, C1606, C603, C604, C605, C606, C703, C704, C705, C706, C803, C804, C805, C806, C903, C904, C905, C906: moved to B.Cu
- R1001, R1002, R1003, R1004, R1101, R1102, R1103, R1104, R1201, R1202, R1203, R1204, R1301, R1302, R1303, R1304, R1401, R1402, R1403, R1404, R1501, R1502, R1503, R1504, R1601, R1602, R1603, R1604, R601, R602, R603, R604, R701, R702, R703, R704, R801, R802, R803, R804, R901, R902, R903, R904: value 75 -> 10k; footprint Capacitors_SMD:C_0603 -> Resistors_SMD:R_0603; moved to B.Cu
- R1701, R1801, R1901: value 10k -> 75; footprint Capacitors_SMD:C_0603 -> Resistors_SMD:R_0603
- R1702, R1802, R1902: footprint Capacitors_SMD:C_0603 -> Resistors_SMD:R_0603
- R1703, R1803, R1903: value 10k -> 75
- R501, R502, R503, R504: value 75 -> 10k; footprint Capacitors_SMD:C_0603 -> Resistors_SMD:R_0603
- moved C805 577.2 mm to (47.6, 115.1)
- moved C804 572.4 mm to (47.6, 122.7)
- moved C803 567.7 mm to (47.6, 130.3)
- moved CONN801 554.9 mm to (52.9, 122.7), turned to 90 degrees
- moved R804 550.6 mm to (60.1, 139.2), turned to 90 degrees
- moved R803 548.2 mm to (58.0, 135.1), turned to 180 degrees
- moved R801 541.6 mm to (60.1, 132.8), turned to 270 degrees
- moved C806 540.7 mm to (58.4, 102.9), turned to 270 degrees
- moved C604 538.2 mm to (22.6, 122.7)
- moved R802 538.1 mm to (59.2, 130.3)
- moved C605 535.3 mm to (22.6, 115.1)
- moved C1103 529.6 mm to (97.6, 62.3)
- moved C802 524.9 mm to (64.9, 142.7), turned to 90 degrees
- moved C606 523.1 mm to (33.4, 102.9), turned to 270 degrees
- moved C1106 516.1 mm to (108.4, 34.9), turned to 270 degrees
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Connections:
- C1001 pad 1: /in-mux/scart_in_6/AO_Right -> /in-mux/scart_in_7/AO_Right
- C1002 pad 1: /in-mux/scart_in_6/AO_Left -> /in-mux/scart_in_7/AO_Left
- C1003 pad 1: /in-mux/scart_in_6/Blue -> /in-mux/scart_in_7/Blue
- C1004 pad 1: /in-mux/scart_in_6/Green -> /in-mux/scart_in_7/Green
- C1005 pad 1: /in-mux/scart_in_6/Red -> /in-mux/scart_in_7/Red
- C1006 pad 1: /in-mux/scart_in_6/Composite -> /in-mux/scart_in_7/Composite
- C1101 pad 1: /in-mux/scart_in_7/AO_Right -> /in-mux/scart_in_8/AO_Right
- C1102 pad 1: /in-mux/scart_in_7/AO_Left -> /in-mux/scart_in_8/AO_Left
- C1103 pad 1: /in-mux/scart_in_7/Blue -> /in-mux/scart_in_8/Blue
- C1104 pad 1: /in-mux/scart_in_7/Green -> /in-mux/scart_in_8/Green
- C1105 pad 1: /in-mux/scart_in_7/Red -> /in-mux/scart_in_8/Red
- C1106 pad 1: /in-mux/scart_in_7/Composite -> /in-mux/scart_in_8/Composite
- C1201 pad 1: /in-mux/scart_in_8/AO_Right -> /in-mux/scart_in_11/AO_Right
- C1202 pad 1: /in-mux/scart_in_8/AO_Left -> /in-mux/scart_in_11/AO_Left
- C1203 pad 1: /in-mux/scart_in_8/Blue -> /in-mux/scart_in_11/Blue
- C1204 pad 1: /in-mux/scart_in_8/Green -> /in-mux/scart_in_11/Green
- C1205 pad 1: /in-mux/scart_in_8/Red -> /in-mux/scart_in_11/Red
- C1206 pad 1: /in-mux/scart_in_8/Composite -> /in-mux/scart_in_11/Composite
- C1301 pad 1: /in-mux/scart_in_11/AO_Right -> /in-mux/scart_in_9/AO_Right
- C1302 pad 1: /in-mux/scart_in_11/AO_Left -> /in-mux/scart_in_9/AO_Left
- C1303 pad 1: /in-mux/scart_in_11/Blue -> /in-mux/scart_in_9/Blue
- C1304 pad 1: /in-mux/scart_in_11/Green -> /in-mux/scart_in_9/Green
- C1305 pad 1: /in-mux/scart_in_11/Red -> /in-mux/scart_in_9/Red
- C1306 pad 1: /in-mux/scart_in_11/Composite -> /in-mux/scart_in_9/Composite
- C1401 pad 1: /in-mux/scart_in_9/AO_Right -> /in-mux/scart_in_12/AO_Right
- C1402 pad 1: /in-mux/scart_in_9/AO_Left -> /in-mux/scart_in_12/AO_Left
- C1403 pad 1: /in-mux/scart_in_9/Blue -> /in-mux/scart_in_12/Blue
- C1404 pad 1: /in-mux/scart_in_9/Green -> /in-mux/scart_in_12/Green
- C1405 pad 1: /in-mux/scart_in_9/Red -> /in-mux/scart_in_12/Red
- C1406 pad 1: /in-mux/scart_in_9/Composite -> /in-mux/scart_in_12/Composite
- C1501 pad 1: /in-mux/scart_in_12/AO_Right -> /in-mux/scart_in_10/AO_Right
- C1502 pad 1: /in-mux/scart_in_12/AO_Left -> /in-mux/scart_in_10/AO_Left
- C1503 pad 1: /in-mux/scart_in_12/Blue -> /in-mux/scart_in_10/Blue
- C1504 pad 1: /in-mux/scart_in_12/Green -> /in-mux/scart_in_10/Green
- C1505 pad 1: /in-mux/scart_in_12/Red -> /in-mux/scart_in_10/Red
- C1506 pad 1: /in-mux/scart_in_12/Composite -> /in-mux/scart_in_10/Composite
- C1601 pad 1: /in-mux/scart_in_10/AO_Right -> /in-mux/scart_in_5/AO_Right
- C1602 pad 1: /in-mux/scart_in_10/AO_Left -> /in-mux/scart_in_5/AO_Left
- C1603 pad 1: /in-mux/scart_in_10/Blue -> /in-mux/scart_in_5/Blue
- C1604 pad 1: /in-mux/scart_in_10/Green -> /in-mux/scart_in_5/Green
- C1605 pad 1: /in-mux/scart_in_10/Red -> /in-mux/scart_in_5/Red
- C1606 pad 1: /in-mux/scart_in_10/Composite -> /in-mux/scart_in_5/Composite
- C901 pad 1: /in-mux/scart_in_5/AO_Right -> /in-mux/scart_in_6/AO_Right
- C902 pad 1: /in-mux/scart_in_5/AO_Left -> /in-mux/scart_in_6/AO_Left
- C903 pad 1: /in-mux/scart_in_5/Blue -> /in-mux/scart_in_6/Blue
- C904 pad 1: /in-mux/scart_in_5/Green -> /in-mux/scart_in_6/Green
- C905 pad 1: /in-mux/scart_in_5/Red -> /in-mux/scart_in_6/Red
- C906 pad 1: /in-mux/scart_in_5/Composite -> /in-mux/scart_in_6/Composite
- CONN1001 pad 1: (no net) -> Net-(CONN1001-Pad1)
- CONN1001 pad 19: (no net) -> Net-(CONN1001-Pad19)
- CONN1001 pad 2: Net-(C1001-Pad2) -> Net-(CONN1001-Pad2)
- CONN1001 pad 3: (no net) -> Net-(CONN1001-Pad3)
- CONN1001 pad 6: Net-(C1002-Pad2) -> Net-(CONN1001-Pad6)
- CONN1101 pad 1: (no net) -> Net-(CONN1101-Pad1)
- CONN1101 pad 19: (no net) -> Net-(CONN1101-Pad19)
- CONN1101 pad 2: Net-(C1101-Pad2) -> Net-(CONN1101-Pad2)
- CONN1101 pad 3: (no net) -> Net-(CONN1101-Pad3)
- CONN1101 pad 6: Net-(C1102-Pad2) -> Net-(CONN1101-Pad6)
- CONN1201 pad 1: (no net) -> Net-(CONN1201-Pad1)
- CONN1201 pad 19: (no net) -> Net-(CONN1201-Pad19)
- CONN1201 pad 2: Net-(C1201-Pad2) -> Net-(CONN1201-Pad2)
- CONN1201 pad 3: (no net) -> Net-(CONN1201-Pad3)
- CONN1201 pad 6: Net-(C1202-Pad2) -> Net-(CONN1201-Pad6)
- CONN1301 pad 1: (no net) -> Net-(CONN1301-Pad1)
- CONN1301 pad 19: (no net) -> Net-(CONN1301-Pad19)
- CONN1301 pad 2: Net-(C1301-Pad2) -> Net-(CONN1301-Pad2)
- CONN1301 pad 3: (no net) -> Net-(CONN1301-Pad3)
- CONN1301 pad 6: Net-(C1302-Pad2) -> Net-(CONN1301-Pad6)
- CONN1401 pad 1: (no net) -> Net-(CONN1401-Pad1)
- CONN1401 pad 19: (no net) -> Net-(CONN1401-Pad19)
- CONN1401 pad 2: Net-(C1401-Pad2) -> Net-(CONN1401-Pad2)
- CONN1401 pad 3: (no net) -> Net-(CONN1401-Pad3)
- CONN1401 pad 6: Net-(C1402-Pad2) -> Net-(CONN1401-Pad6)
- CONN1501 pad 1: (no net) -> Net-(CONN1501-Pad1)
- CONN1501 pad 19: (no net) -> Net-(CONN1501-Pad19)
- CONN1501 pad 2: Net-(C1501-Pad2) -> Net-(CONN1501-Pad2)
- CONN1501 pad 3: (no net) -> Net-(CONN1501-Pad3)
- CONN1501 pad 6: Net-(C1502-Pad2) -> Net-(CONN1501-Pad6)
- CONN1601 pad 1: (no net) -> Net-(CONN1601-Pad1)
- CONN1601 pad 19: (no net) -> Net-(CONN1601-Pad19)
- CONN1601 pad 2: Net-(C1601-Pad2) -> Net-(CONN1601-Pad2)
- CONN1601 pad 3: (no net) -> Net-(CONN1601-Pad3)
- CONN1601 pad 6: Net-(C1602-Pad2) -> Net-(CONN1601-Pad6)
- CONN1701 pad 1: Net-(CONN1701-Pad1) -> Net-(C1701-Pad2)
- CONN1701 pad 19: Net-(CONN1701-Pad19) -> /scart_out_1/C
- CONN1701 pad 3: Net-(CONN1701-Pad3) -> Net-(C1702-Pad2)
- CONN1801 pad 1: Net-(CONN1801-Pad1) -> Net-(C1801-Pad2)
- CONN1801 pad 19: Net-(CONN1801-Pad19) -> /scart_out_2/C
- CONN1801 pad 3: Net-(CONN1801-Pad3) -> Net-(C1802-Pad2)
- CONN1901 pad 1: Net-(CONN1901-Pad1) -> Net-(C1901-Pad2)
- CONN1901 pad 19: Net-(CONN1901-Pad19) -> /scart_out_3/C
- CONN1901 pad 3: Net-(CONN1901-Pad3) -> Net-(C1902-Pad2)
- CONN501 pad 1: (no net) -> Net-(CONN501-Pad1)
- CONN501 pad 19: (no net) -> Net-(CONN501-Pad19)
- CONN501 pad 2: Net-(C501-Pad2) -> Net-(CONN501-Pad2)
- CONN501 pad 3: (no net) -> Net-(CONN501-Pad3)
- CONN501 pad 6: Net-(C502-Pad2) -> Net-(CONN501-Pad6)
- CONN601 pad 1: (no net) -> Net-(CONN601-Pad1)
- CONN601 pad 19: (no net) -> Net-(CONN601-Pad19)
- CONN601 pad 2: Net-(C601-Pad2) -> Net-(CONN601-Pad2)
- CONN601 pad 3: (no net) -> Net-(CONN601-Pad3)
- CONN601 pad 6: Net-(C602-Pad2) -> Net-(CONN601-Pad6)
- CONN701 pad 1: (no net) -> Net-(CONN701-Pad1)
- CONN701 pad 19: (no net) -> Net-(CONN701-Pad19)
- CONN701 pad 2: Net-(C701-Pad2) -> Net-(CONN701-Pad2)
- CONN701 pad 3: (no net) -> Net-(CONN701-Pad3)
- CONN701 pad 6: Net-(C702-Pad2) -> Net-(CONN701-Pad6)
- CONN801 pad 1: (no net) -> Net-(CONN801-Pad1)
- CONN801 pad 19: (no net) -> Net-(CONN801-Pad19)
- CONN801 pad 2: Net-(C801-Pad2) -> Net-(CONN801-Pad2)
- CONN801 pad 3: (no net) -> Net-(CONN801-Pad3)
- CONN801 pad 6: Net-(C802-Pad2) -> Net-(CONN801-Pad6)
- CONN901 pad 1: (no net) -> Net-(CONN901-Pad1)
- CONN901 pad 19: (no net) -> Net-(CONN901-Pad19)
- CONN901 pad 2: Net-(C901-Pad2) -> Net-(CONN901-Pad2)
- CONN901 pad 3: (no net) -> Net-(CONN901-Pad3)
- CONN901 pad 6: Net-(C902-Pad2) -> Net-(CONN901-Pad6)
- GS1701 pad 3: Net-(CONN1701-Pad1) -> Net-(C1701-Pad2)
- GS1702 pad 3: Net-(CONN1701-Pad3) -> Net-(C1702-Pad2)
- GS1703 pad 3: Net-(CONN1701-Pad19) -> /scart_out_1/C
- GS1801 pad 3: Net-(CONN1801-Pad1) -> Net-(C1801-Pad2)
- GS1802 pad 3: Net-(CONN1801-Pad3) -> Net-(C1802-Pad2)
- GS1803 pad 3: Net-(CONN1801-Pad19) -> /scart_out_2/C
- GS1901 pad 3: Net-(CONN1901-Pad1) -> Net-(C1901-Pad2)
- GS1902 pad 3: Net-(CONN1901-Pad3) -> Net-(C1902-Pad2)
- GS1903 pad 3: Net-(CONN1901-Pad19) -> /scart_out_3/C
- IC301 pad 25: (no net) -> /micro/LED_R
- IC301 pad 26: (no net) -> /micro/LED_G
- P101 pad 1: (no net) -> /psus/VBUS
- P101 pad 5: /psus/GNDIN -> GND
- P101 pad 6: /psus/GNDIN -> GND
- R1001 pad 1: Net-(C1003-Pad2) -> Net-(R1001-Pad1)
- R1001 pad 2: GND -> Net-(C1001-Pad2)
- R1002 pad 1: Net-(C1004-Pad2) -> Net-(CONN1001-Pad6)
- R1002 pad 2: GND -> Net-(R1001-Pad1)
- R1003 pad 1: Net-(C1005-Pad2) -> Net-(C1001-Pad2)
- R1004 pad 1: Net-(C1006-Pad2) -> Net-(R1004-Pad1)
- R1004 pad 2: GND -> Net-(C1002-Pad2)
- R1101 pad 1: Net-(C1103-Pad2) -> Net-(R1101-Pad1)
- R1101 pad 2: GND -> Net-(C1101-Pad2)
- R1102 pad 1: Net-(C1104-Pad2) -> Net-(CONN1101-Pad6)
- R1102 pad 2: GND -> Net-(R1101-Pad1)
- R1103 pad 1: Net-(C1105-Pad2) -> Net-(C1101-Pad2)
- R1104 pad 1: Net-(C1106-Pad2) -> Net-(R1104-Pad1)
- R1104 pad 2: GND -> Net-(C1102-Pad2)
- R1201 pad 1: Net-(C1203-Pad2) -> Net-(R1201-Pad1)
- R1201 pad 2: GND -> Net-(C1201-Pad2)
- R1202 pad 1: Net-(C1204-Pad2) -> Net-(CONN1201-Pad6)
- R1202 pad 2: GND -> Net-(R1201-Pad1)
- R1203 pad 1: Net-(C1205-Pad2) -> Net-(C1201-Pad2)
- R1204 pad 1: Net-(C1206-Pad2) -> Net-(R1204-Pad1)
- R1204 pad 2: GND -> Net-(C1202-Pad2)
- R1301 pad 1: Net-(C1303-Pad2) -> Net-(R1301-Pad1)
- R1301 pad 2: GND -> Net-(C1301-Pad2)
- R1302 pad 1: Net-(C1304-Pad2) -> Net-(CONN1301-Pad6)
- R1302 pad 2: GND -> Net-(R1301-Pad1)
- R1303 pad 1: Net-(C1305-Pad2) -> Net-(C1301-Pad2)
- R1304 pad 1: Net-(C1306-Pad2) -> Net-(R1304-Pad1)
- R1304 pad 2: GND -> Net-(C1302-Pad2)
- R1401 pad 1: Net-(C1403-Pad2) -> Net-(R1401-Pad1)
- R1401 pad 2: GND -> Net-(C1401-Pad2)
- R1402 pad 1: Net-(C1404-Pad2) -> Net-(CONN1401-Pad6)
- R1402 pad 2: GND -> Net-(R1401-Pad1)
- R1403 pad 1: Net-(C1405-Pad2) -> Net-(C1401-Pad2)
- R1404 pad 1: Net-(C1406-Pad2) -> Net-(R1404-Pad1)
- R1404 pad 2: GND -> Net-(C1402-Pad2)
- R1501 pad 1: Net-(C1503-Pad2) -> Net-(R1501-Pad1)
- R1501 pad 2: GND -> Net-(C1501-Pad2)
- R1502 pad 1: Net-(C1504-Pad2) -> Net-(CONN1501-Pad6)
- R1502 pad 2: GND -> Net-(R1501-Pad1)
- R1503 pad 1: Net-(C1505-Pad2) -> Net-(C1501-Pad2)
- R1504 pad 1: Net-(C1506-Pad2) -> Net-(R1504-Pad1)
- R1504 pad 2: GND -> Net-(C1502-Pad2)
- R1601 pad 1: Net-(C1603-Pad2) -> Net-(R1601-Pad1)
- R1601 pad 2: GND -> Net-(C1601-Pad2)
- R1602 pad 1: Net-(C1604-Pad2) -> Net-(CONN1601-Pad6)
- R1602 pad 2: GND -> Net-(R1601-Pad1)
- R1603 pad 1: Net-(C1605-Pad2) -> Net-(C1601-Pad2)
- R1604 pad 1: Net-(C1606-Pad2) -> Net-(R1604-Pad1)
- R1604 pad 2: GND -> Net-(C1602-Pad2)
- R1701 pad 1: +12V -> Net-(C1701-Pad2)
- R1701 pad 2: Net-(Q1701-Pad1) -> GND
- R1702 pad 1: /scart_out_1/RGB -> Net-(C1702-Pad2)
- R1702 pad 2: Net-(CONN1701-Pad16) -> GND
- R1703 pad 1: /scart_out_1/ASPECT -> /scart_out_1/RGB
- R1703 pad 2: Net-(Q1703-Pad1) -> Net-(CONN1701-Pad16)
- R1801 pad 1: +12V -> Net-(C1801-Pad2)
- R1801 pad 2: Net-(Q1801-Pad1) -> GND
- R1802 pad 1: /scart_out_2/RGB -> Net-(C1802-Pad2)
- R1802 pad 2: Net-(CONN1801-Pad16) -> GND
- R1803 pad 1: /scart_out_2/ASPECT -> /scart_out_2/RGB
- R1803 pad 2: Net-(Q1803-Pad1) -> Net-(CONN1801-Pad16)
- R1901 pad 1: +12V -> Net-(C1901-Pad2)
- R1901 pad 2: Net-(Q1901-Pad1) -> GND
- R1902 pad 1: (no net) -> Net-(C1902-Pad2)
- R1902 pad 2: Net-(CONN1901-Pad16) -> GND
- R1903 pad 1: /scart_out_3/ASPECT -> (no net)
- R1903 pad 2: Net-(Q1903-Pad1) -> Net-(CONN1901-Pad16)
- R303 pad 1: (no net) -> Net-(D301-Pad4)
- R304 pad 1: (no net) -> Net-(D301-Pad2)
- R501 pad 1: Net-(C503-Pad2) -> Net-(R501-Pad1)
- R501 pad 2: GND -> Net-(C501-Pad2)
- R502 pad 1: Net-(C504-Pad2) -> Net-(CONN501-Pad6)
- R502 pad 2: GND -> Net-(R501-Pad1)
- R503 pad 1: Net-(C505-Pad2) -> Net-(C501-Pad2)
- R504 pad 1: Net-(C506-Pad2) -> Net-(R504-Pad1)
- R504 pad 2: GND -> Net-(C502-Pad2)
- R601 pad 1: Net-(C603-Pad2) -> Net-(R601-Pad1)
- R601 pad 2: GND -> Net-(C601-Pad2)
- R602 pad 1: Net-(C604-Pad2) -> Net-(CONN601-Pad6)
- R602 pad 2: GND -> Net-(R601-Pad1)
- R603 pad 1: Net-(C605-Pad2) -> Net-(C601-Pad2)
- R604 pad 1: Net-(C606-Pad2) -> Net-(R604-Pad1)
- R604 pad 2: GND -> Net-(C602-Pad2)
- R701 pad 1: Net-(C703-Pad2) -> Net-(R701-Pad1)
- R701 pad 2: GND -> Net-(C701-Pad2)
- R702 pad 1: Net-(C704-Pad2) -> Net-(CONN701-Pad6)
- R702 pad 2: GND -> Net-(R701-Pad1)
- R703 pad 1: Net-(C705-Pad2) -> Net-(C701-Pad2)
- R704 pad 1: Net-(C706-Pad2) -> Net-(R704-Pad1)
- R704 pad 2: GND -> Net-(C702-Pad2)
- R801 pad 1: Net-(C803-Pad2) -> Net-(R801-Pad1)
- R801 pad 2: GND -> Net-(C801-Pad2)
- R802 pad 1: Net-(C804-Pad2) -> Net-(CONN801-Pad6)
- R802 pad 2: GND -> Net-(R801-Pad1)
- R803 pad 1: Net-(C805-Pad2) -> Net-(C801-Pad2)
- R804 pad 1: Net-(C806-Pad2) -> Net-(R804-Pad1)
- R804 pad 2: GND -> Net-(C802-Pad2)
- R901 pad 1: Net-(C903-Pad2) -> Net-(R901-Pad1)
- R901 pad 2: GND -> Net-(C901-Pad2)
- R902 pad 1: Net-(C904-Pad2) -> Net-(CONN901-Pad6)
- R902 pad 2: GND -> Net-(R901-Pad1)
- R903 pad 1: Net-(C905-Pad2) -> Net-(C901-Pad2)
- R904 pad 1: Net-(C906-Pad2) -> Net-(R904-Pad1)
- R904 pad 2: GND -> Net-(C902-Pad2)
Routing:
- net GND: track 20.8 -> 241.3 mm
- net Net-(C1406-Pad2): track 0.00 -> 22.4 mm
- net Net-(C1306-Pad2): track 0.00 -> 22.4 mm
- net Net-(C1206-Pad2): track 0.00 -> 22.4 mm
- net Net-(C1006-Pad2): track 0.00 -> 22.4 mm
- net Net-(C606-Pad2): track 0.00 -> 22.4 mm
- net Net-(C1606-Pad2): track 0.00 -> 22.4 mm
- net Net-(C906-Pad2): track 0.00 -> 22.4 mm
- net Net-(C806-Pad2): track 0.00 -> 22.4 mm
- net Net-(C1106-Pad2): track 0.00 -> 22.4 mm
- net Net-(C1506-Pad2): track 0.00 -> 22.4 mm
- net Net-(C706-Pad2): track 0.00 -> 22.4 mm
- net Net-(CONN1201-Pad2): track 0.00 -> 19.9 mm
- net Net-(CONN1001-Pad2): track 0.00 -> 19.9 mm
- net Net-(CONN801-Pad2): track 0.00 -> 19.9 mm
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Other:
- net class Default: clearance 0.254 -> 0.1524; trace_width 0.508 -> 0.254
- rule pad_to_mask_clearance: 0.2 -> 0
- rule trace_clearance: 0.254 -> 0.1524
- rule trace_min: 0.0889 -> 0.2
- rule via_min_drill: 0.2 -> 0.3
- rule via_min_size: 0.45 -> 0.4

Commit message: + Start the layout * (switching to new OS so need to push this!)
Parts:
- moved R407 404.3 mm to (191.0, 62.9), turned to 180 degrees
- moved R402 403.5 mm to (191.0, 43.3), turned to 180 degrees
- moved R406 403.4 mm to (191.0, 44.9), turned to 180 degrees
- moved C408 401.9 mm to (179.9, 47.7), turned to 270 degrees
- moved R403 400.4 mm to (191.0, 61.3), turned to 180 degrees
- moved C424 400.3 mm to (179.9, 119.7), turned to 270 degrees
- moved R404 398.8 mm to (191.0, 79.3), turned to 180 degrees
- moved C406 398.6 mm to (178.3, 47.7), turned to 270 degrees
- moved C410 397.2 mm to (178.3, 65.7), turned to 270 degrees
- moved C405 397.0 mm to (191.8, 48.8), turned to 270 degrees
- moved R413 396.6 mm to (191.0, 97.3), turned to 180 degrees
- moved C423 394.3 mm to (190.2, 120.8), turned to 270 degrees
- moved R410 394.1 mm to (191.0, 46.5), turned to 180 degrees
- moved R411 393.8 mm to (191.0, 64.5), turned to 180 degrees
- moved C422 393.2 mm to (178.3, 119.7), turned to 270 degrees
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Connections:
- U401 pad 10: /in-mux/scart_in_8/Red -> /in-mux/scart_in_4/Red
- U401 pad 11: /in-mux/scart_in_9/Red -> /in-mux/scart_in_7/Red
- U401 pad 12: /in-mux/scart_in_10/Red -> /in-mux/scart_in_11/Red
- U401 pad 13: /in-mux/scart_in_11/Red -> /in-mux/scart_in_12/Red
- U401 pad 14: /in-mux/scart_in_12/Red -> /in-mux/scart_in_5/Red
- U401 pad 2: /in-mux/scart_in_2/Red -> /in-mux/scart_in_3/Red
- U401 pad 3: /in-mux/scart_in_3/Red -> /in-mux/scart_in_6/Red
- U401 pad 4: /in-mux/scart_in_4/Red -> /in-mux/scart_in_8/Red
- U401 pad 5: /in-mux/scart_in_5/Red -> /in-mux/scart_in_9/Red
- U401 pad 6: /in-mux/scart_in_6/Red -> /in-mux/scart_in_10/Red
- U401 pad 9: /in-mux/scart_in_7/Red -> /in-mux/scart_in_2/Red
- U402 pad 10: /in-mux/scart_in_8/Green -> /in-mux/scart_in_11/Green
- U402 pad 12: /in-mux/scart_in_10/Green -> /in-mux/scart_in_12/Green
- U402 pad 13: /in-mux/scart_in_11/Green -> /in-mux/scart_in_10/Green
- U402 pad 14: /in-mux/scart_in_12/Green -> /in-mux/scart_in_5/Green
- U402 pad 5: /in-mux/scart_in_5/Green -> /in-mux/scart_in_6/Green
- U402 pad 6: /in-mux/scart_in_6/Green -> /in-mux/scart_in_7/Green
- U402 pad 9: /in-mux/scart_in_7/Green -> /in-mux/scart_in_8/Green
- U403 pad 10: /in-mux/scart_in_8/Blue -> /in-mux/scart_in_11/Blue
- U403 pad 12: /in-mux/scart_in_10/Blue -> /in-mux/scart_in_12/Blue
- U403 pad 13: /in-mux/scart_in_11/Blue -> /in-mux/scart_in_10/Blue
- U403 pad 14: /in-mux/scart_in_12/Blue -> /in-mux/scart_in_5/Blue
- U403 pad 5: /in-mux/scart_in_5/Blue -> /in-mux/scart_in_6/Blue
- U403 pad 6: /in-mux/scart_in_6/Blue -> /in-mux/scart_in_7/Blue
- U403 pad 9: /in-mux/scart_in_7/Blue -> /in-mux/scart_in_8/Blue
- U404 pad 10: /in-mux/scart_in_8/Composite -> /in-mux/scart_in_11/Composite
- U404 pad 12: /in-mux/scart_in_10/Composite -> /in-mux/scart_in_12/Composite
- U404 pad 13: /in-mux/scart_in_11/Composite -> /in-mux/scart_in_10/Composite
- U404 pad 14: /in-mux/scart_in_12/Composite -> /in-mux/scart_in_5/Composite
- U404 pad 5: /in-mux/scart_in_5/Composite -> /in-mux/scart_in_6/Composite
- U404 pad 6: /in-mux/scart_in_6/Composite -> /in-mux/scart_in_7/Composite
- U404 pad 9: /in-mux/scart_in_7/Composite -> /in-mux/scart_in_8/Composite
- U405 pad 10: /in-mux/scart_in_8/AO_Right -> /in-mux/scart_in_11/AO_Right
- U405 pad 12: /in-mux/scart_in_10/AO_Right -> /in-mux/scart_in_12/AO_Right
- U405 pad 13: /in-mux/scart_in_11/AO_Right -> /in-mux/scart_in_10/AO_Right
- U405 pad 14: /in-mux/scart_in_12/AO_Right -> /in-mux/scart_in_5/AO_Right
- U405 pad 5: /in-mux/scart_in_5/AO_Right -> /in-mux/scart_in_6/AO_Right
- U405 pad 6: /in-mux/scart_in_6/AO_Right -> /in-mux/scart_in_7/AO_Right
- U405 pad 9: /in-mux/scart_in_7/AO_Right -> /in-mux/scart_in_8/AO_Right
- U406 pad 10: /in-mux/scart_in_8/AO_Left -> /in-mux/scart_in_11/AO_Left
- U406 pad 12: /in-mux/scart_in_10/AO_Left -> /in-mux/scart_in_12/AO_Left
- U406 pad 13: /in-mux/scart_in_11/AO_Left -> /in-mux/scart_in_10/AO_Left
- U406 pad 14: /in-mux/scart_in_12/AO_Left -> /in-mux/scart_in_5/AO_Left
- U406 pad 5: /in-mux/scart_in_5/AO_Left -> /in-mux/scart_in_6/AO_Left
- U406 pad 6: /in-mux/scart_in_6/AO_Left -> /in-mux/scart_in_7/AO_Left
- U406 pad 9: /in-mux/scart_in_7/AO_Left -> /in-mux/scart_in_8/AO_Left
Routing:
- net /in-mux/scart_in_1/Red: track 0.00 -> 181.3 mm, vias 0 -> 1
- net /in-mux/scart_in_3/Red: track 0.00 -> 155.3 mm, vias 0 -> 1
- net /in-mux/scart_in_6/Red: track 0.00 -> 130.0 mm, vias 0 -> 1
- net /in-mux/scart_in_8/Red: track 0.00 -> 103.0 mm, vias 0 -> 1
- net /in-mux/scart_in_9/Red: track 0.00 -> 79.0 mm, vias 0 -> 1
- net GND: track 241.3 -> 314.9 mm
- net +5VA: track 14.0 -> 83.7 mm
- net /in-mux/scart_in_10/Red: track 0.00 -> 52.4 mm, vias 0 -> 1
- net Net-(R418-Pad2): track 0.00 -> 2.58 mm
- net Net-(R417-Pad2): track 0.00 -> 2.58 mm
- net Net-(R412-Pad2): track 0.00 -> 2.58 mm
- net Net-(R411-Pad2): track 0.00 -> 2.58 mm
- net Net-(R410-Pad2): track 0.00 -> 2.58 mm
- net Net-(R403-Pad2): track 0.00 -> 2.47 mm
- net Net-(R402-Pad2): track 0.00 -> 2.47 mm
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